File: MX3-11-8/Protoboard MX3-11-8.sch (EAGLE design)
At the start: 719 parts, among them J1 DCJ0202

Commit message: Update Gerb files
Created Gerber files for MX 2-7-6 without ESP
Parts:
- added JP1: USB-RECEPTABLE, daspilker:USB-RECEPTABLE
- added U1: 3.3V/150mA, SparkFun-PowerIC:V_REG_MIC52053.3V
Connections:
- net GND: now also JP1.GND, U1.GND
- net VCC: now also JP1.VCC, U1.EN, U1.IN
- net VDD: now also U1.OUT
Changed lines of the file:
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@@
 <?xml version="1.0" encoding="utf-8"?>
 <!DOCTYPE eagle SYSTEM "eagle.dtd">
-<eagle version="7.6.0">
+<eagle version="7.7.0">
 <drawing>
 <settings>
@@
 <part name="PAD254" library="wirepad" deviceset="1,6/0,8" device=""/>
 <part name="PAD255" library="wirepad" deviceset="1,6/0,8" device=""/>
+<part name="U1" library="SparkFun-PowerIC" deviceset="V_REG_MIC5205" device="3.3V" value="3.3V/150mA"/>
+<part name="JP1" library="daspilker" deviceset="USB-RECEPTABLE" device=""/>
+<part name="SUPPLY1" library="supply2" deviceset="VCC" device=""/>
+<part name="GND5" library="supply1" deviceset="GND" device=""/>
+<part name="VDD4" library="supply1" deviceset="VDD" device=""/>
+<part name="SUPPLY2" library="supply2" deviceset="VCC" device=""/>
+<part name="GND6" library="supply1" deviceset="GND" device=""/>
 </parts>
 <sheets>
@@
 <attribute name="VALUE" x="245.237" y="-13.462" size="1.778" layer="96"/>
 </instance>
+<instance part="U1" gate="U1" x="-25.4" y="88.9"/>
+<instance part="JP1" gate="G$1" x="-40.64" y="30.48"/>
+<instance part="SUPPLY1" gate="G$1" x="-43.18" y="99.06"/>
+<instance part="GND5" gate="1" x="-43.18" y="78.74"/>
+<instance part="VDD4" gate="G$1" x="-10.16" y="99.06"/>
+<instance part="SUPPLY2" gate="G$1" x="-53.34" y="40.64"/>
+<instance part="GND6" gate="1" x="-53.34" y="17.78"/>
 </instances>
 <busses>
@@
 <wire x1="50.8" y1="35.56" x2="50.8" y2="40.64" width="0.1524" layer="91"/>
 </segment>
+<segment>
+<pinref part="JP1" gate="G$1" pin="GND"/>
+<pinref part="GND6" gate="1" pin="GND"/>
+<wire x1="-48.26" y1="25.4" x2="-53.34" y2="25.4" width="0.1524" layer="91"/>
+<wire x1="-53.34" y1="25.4" x2="-53.34" y2="20.32" width="0.1524" layer="91"/>
+</segment>
+<segment>
+<pinref part="U1" gate="U1" pin="GND"/>
+<pinref part="GND5" gate="1" pin="GND"/>
+<wire x1="-35.56" y1="83.82" x2="-43.18" y2="83.82" width="0.1524" layer="91"/>
+<wire x1="-43.18" y1="83.82" x2="-43.18" y2="81.28" width="0.1524" layer="91"/>
+</segment>
 </net>
 <net name="VCC" class="0">
@@
 <wire x1="-45.72" y1="63.5" x2="-40.64" y2="63.5" width="0.1524" layer="91"/>
 </segment>
+<segment>
+<pinref part="JP1" gate="G$1" pin="VCC"/>
+<pinref part="SUPPLY2" gate="G$1" pin="VCC"/>
+<wire x1="-48.26" y1="35.56" x2="-53.34" y2="35.56" width="0.1524" layer="91"/>
+<wire x1="-53.34" y1="35.56" x2="-53.34" y2="38.1" width="0.1524" layer="91"/>
+</segment>
+<segment>
+<pinref part="U1" gate="U1" pin="EN"/>
+<pinref part="SUPPLY1" gate="G$1" pin="VCC"/>
+<wire x1="-35.56" y1="88.9" x2="-43.18" y2="88.9" width="0.1524" layer="91"/>
+<wire x1="-43.18" y1="88.9" x2="-43.18" y2="93.98" width="0.1524" layer="91"/>
+<pinref part="U1" gate="U1" pin="IN"/>
+<wire x1="-43.18" y1="93.98" x2="-43.18" y2="96.52" width="0.1524" layer="91"/>
+<wire x1="-35.56" y1="93.98" x2="-43.18" y2="93.98" width="0.1524" layer="91"/>
+<junction x="-43.18" y="93.98"/>
+</segment>
 </net>
 <net name="N$1" class="0">
@@
 <wire x1="25.4" y1="45.72" x2="25.4" y2="50.8" width="0.1524" layer="91"/>
 </segment>
+<segment>
+<pinref part="U1" gate="U1" pin="OUT"/>
+<pinref part="VDD4" gate="G$1" pin="VDD"/>
+<wire x1="-17.78" y1="93.98" x2="-10.16" y2="93.98" width="0.1524" layer="91"/>
+<wire x1="-10.16" y1="93.98" x2="-10.16" y2="96.52" width="0.1524" layer="91"/>
+</segment>
 </net>

Commit message: Update to rev2
Updated to Pin headers instead of single wire pads
Parts:
- removed 1, 2, 3, 4, 5, 6, 7, 8, PAD1, PAD10, PAD100, PAD101, PAD102, PAD103, PAD104, PAD105, PAD106, PAD107, PAD108, PAD109, PAD11, PAD110, PAD111, PAD112, PAD113, PAD114, PAD115, PAD116, PAD117, PAD118, PAD119, PAD12, PAD120, PAD121, PAD122, PAD123, PAD124, PAD125, PAD126, PAD127, PAD128, PAD129, PAD13, PAD130, PAD131, PAD132, PAD133, PAD134, PAD135, PAD136, PAD137, PAD138, PAD139, PAD14, PAD140, PAD141, PAD142, PAD143, PAD144, PAD145, PAD146, PAD147, PAD148, PAD149, PAD15, PAD150, PAD151, PAD152, PAD153, PAD154, PAD155, PAD156, PAD157, PAD158, PAD159, PAD16, PAD160, PAD161, PAD162, PAD163, PAD164, PAD165, PAD166, PAD167, PAD168, PAD169, PAD17, PAD170, PAD171, PAD172, PAD173, PAD174, PAD175, PAD176, PAD177, PAD178, PAD179, PAD18, PAD180, PAD181, PAD182, PAD183, PAD184, PAD185, PAD186, PAD187, PAD188, PAD189, PAD19, PAD190, PAD191, PAD192, PAD193, PAD194, PAD195, PAD196, PAD197, PAD198, PAD199, PAD2, PAD20, PAD200, PAD201, PAD202, PAD203, PAD204, PAD205, PAD206, PAD207, PAD208, PAD209, PAD21, PAD210, PAD211, PAD212, PAD213, PAD214, PAD215, PAD216, PAD217, PAD218, PAD219, PAD22, PAD220, PAD221, PAD222, PAD223, PAD224, PAD225, PAD226, PAD227, PAD228, PAD229, PAD23, PAD230, PAD231, PAD232, PAD233, PAD234, PAD235, PAD236, PAD237, PAD238, PAD239, PAD24, PAD240, PAD249, PAD25, PAD250, PAD251, PAD252, PAD253, PAD254, PAD255, PAD26, PAD260, PAD261, PAD262, PAD263, PAD264, PAD265, PAD266, PAD269, PAD27, PAD270, PAD271, PAD272, PAD273, PAD274, PAD275, PAD276, PAD277, PAD278, PAD279, PAD28, PAD280, PAD281, PAD282, PAD283, PAD284, PAD285, PAD286, PAD287, PAD288, PAD289, PAD29, PAD290, PAD291, PAD292, PAD293, PAD294, PAD295, PAD296, PAD297, PAD298, PAD299, PAD3, PAD30, PAD300, PAD301, PAD302, PAD303, PAD304, PAD305, PAD306, PAD307, PAD308, PAD309, PAD31, PAD310, PAD311, PAD312, PAD313, PAD314, PAD315, PAD316, PAD317, PAD318, PAD319, PAD32, PAD320, PAD321, PAD322, PAD323, PAD324, PAD325, PAD326, PAD327, PAD328, PAD329, PAD33, PAD330, PAD331, PAD332, PAD333, PAD334, PAD335, PAD336, PAD337, PAD338, PAD339, PAD34, PAD340, PAD341, PAD342, PAD343, PAD344, PAD345, PAD346, PAD347, PAD348, PAD349, PAD35, PAD350, PAD351, PAD352, PAD353, PAD354, PAD355, PAD356, PAD357, PAD358, PAD359, PAD36, PAD360, PAD361, PAD362, PAD363, PAD364, PAD365, PAD366, PAD367, PAD368, PAD369, PAD37, PAD370, PAD371, PAD372, PAD373, PAD374, PAD375, PAD376, PAD377, PAD378, PAD379, PAD38, PAD380, PAD381, PAD382, PAD383, PAD384, PAD385, PAD386, PAD387, PAD388, PAD389, PAD39, PAD390, PAD391, PAD392, PAD393, PAD394, PAD395, PAD4, PAD40, PAD41, PAD414, PAD415, PAD416, PAD42, PAD420, PAD421, PAD422, PAD423, PAD424, PAD425, PAD426, PAD427, PAD428, PAD429, PAD43, PAD430, PAD431, PAD432, PAD433, PAD434, PAD435, PAD436, PAD437, PAD438, PAD439, PAD44, PAD440, PAD441, PAD442, PAD443, PAD444, PAD445, PAD446, PAD447, PAD448, PAD449, PAD45, PAD450, PAD451, PAD452, PAD453, PAD454, PAD455, PAD456, PAD457, PAD458, PAD459, PAD46, PAD460, PAD461, PAD462, PAD463, PAD464, PAD465, PAD466, PAD467, PAD468, PAD469, PAD47, PAD470, PAD471, PAD472, PAD473, PAD474, PAD475, PAD476, PAD477, PAD478, PAD479, PAD48, PAD480, PAD481, PAD482, PAD483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: (no value), wirepad:1,6/0,8
- removed PAD241, PAD242, PAD243, PAD244, PAD245, PAD246, PAD247, PAD248, PAD734, PAD735, PAD736, PAD737, PAD738, PAD739, PAD740, PAD741, PAD750, PAD751, PAD752, PAD753, PAD754, PAD755, PAD756, PAD757: (no value), wirepad:3,17/1,3
- added J10, J11, J12, J13, J14, J15, J16, J17, J18, J19, J2, J20, J21, J22, J23, J3, J4, J5, J6, J7, J8, J9: (no value), SparkFun-Connectors:M06NO_SILK_FEMALE_PTH
- added J24, J25, J26, J27, J28, J29, J30, J31, J32, J33, J34, J35, J36, J37, J38, J39, J40, J41, J42, J43, J44, J45, J46, J47, J48, J49, J50, J51, J52, J53, J54, J55, J56, J57, J58, J59, J60, J61, J62, J63, J64, J65, J66, J67, J68, J69, J70, J71, J72, J73, J74, J75, J76, J77, J78, J79, J80, J81, J82, J83, J84, J85, J86, J87, J88: (no value), SparkFun-Connectors:M07NO_SILK
- added J89: (no value), SparkFun-Connectors:M04NO_SILK_ALL_ROUND
- added J90, J91, J92, J93: (no value), SparkFun-Connectors:M20NO_SILK_KIT
- added JP10, JP11, JP12, JP13, JP14, JP15, JP16, JP17, JP18, JP19, JP20, JP21, JP22, JP23, JP24, JP25: (no value), adafruit:PINHD-1X1CB
- added JP2, JP3, JP4, JP5, JP6, JP7, JP8, JP9: (no value), adafruit:PINHD-1X1-BIGPOGO
Connections:
- removed net N$100: PAD699.P, PAD700.P, PAD701.P, PAD702.P, PAD703.P, PAD704.P, PAD705.P
- removed net N$101: PAD706.P, PAD707.P, PAD708.P, PAD709.P, PAD710.P, PAD711.P, PAD712.P
- removed net N$102: 1.P, RJ-1-1.P
- removed net N$103: 2.P, RJ-2-1.P
- removed net N$104: 3.P, RJ-3.P
- removed net N$105: 4.P, RJ-4-1.P
- removed net N$106: 5.P, RJ-5-1.P
- removed net N$107: 6.P, RJ-6-1.P
- removed net N$108: 7.P, RJ-7-1.P
- removed net N$109: 8.P, RJ-8-1.P
- removed net N$110: PAD713.P, PAD714.P, PAD715.P, PAD716.P, PAD717.P, PAD718.P, PAD719.P
- removed net N$111: PAD720.P, PAD721.P, PAD722.P, PAD723.P, PAD724.P, PAD725.P, PAD726.P
- removed net N$112: PAD727.P, PAD728.P, PAD729.P, PAD730.P, PAD731.P, PAD732.P, PAD733.P
- removed net N$113: PAD734.P, PAD757.P
- removed net N$114: PAD735.P, PAD756.P
- removed net N$115: PAD736.P, PAD755.P
- removed net N$116: PAD737.P, PAD754.P
- removed net N$117: PAD738.P, PAD753.P
- removed net N$118: PAD739.P, PAD752.P
- removed net N$119: PAD740.P, PAD751.P
- removed net N$120: PAD741.P, PAD750.P
- removed net N$97: PAD678.P, PAD679.P, PAD680.P, PAD681.P, PAD682.P, PAD683.P, PAD684.P
- removed net N$98: PAD685.P, PAD686.P, PAD687.P, PAD688.P, PAD689.P, PAD690.P, PAD691.P
- removed net N$99: PAD692.P, PAD693.P, PAD694.P, PAD695.P, PAD696.P, PAD697.P, PAD698.P
- new net N$47: J48.1, J48.2, J48.3, J48.4, J48.5, J48.6, J48.7
- new net N$48: J49.1, J49.2, J49.3, J49.4, J49.5, J49.6, J49.7
- new net N$52: J53.1, J53.2, J53.3, J53.4, J53.5, J53.6, J53.7
- new net N$53: J54.1, J54.2, J54.3, J54.4, J54.5, J54.6, J54.7
- new net N$54: J55.1, J55.2, J55.3, J55.4, J55.5, J55.6, J55.7
- new net N$55: J56.1, J56.2, J56.3, J56.4, J56.5, J56.6, J56.7
- new net N$56: J57.1, J57.2, J57.3, J57.4, J57.5, J57.6, J57.7
- new net N$57: J58.1, J58.2, J58.3, J58.4, J58.5, J58.6, J58.7
- new net N$58: J59.1, J59.2, J59.3, J59.4, J59.5, J59.6, J59.7
- new net N$85: J86.1, J86.2, J86.3, J86.4, J86.5, J86.6, J86.7
- new net N$86: J87.1, J87.2, J87.3, J87.4, J87.5, J87.6, J87.7
- new net N$87: J88.1, J88.2, J88.3, J88.4, J88.5, J88.6, J88.7
- new net N$88: J89.1, J89.2, J89.3, J89.4
- new net N$89: JP10.1, JP2.1
- new net N$90: JP11.1, JP3.1
- new net N$91: JP12.1, JP4.1
- net GND: now also J91.1, J91.10, J91.11, J91.12, J91.13, J91.14, J91.15, J91.16, J91.17, J91.18, J91.19, J91.2, J91.20, J91.3, J91.4, J91.5, J91.6, J91.7, J91.8, J91.9, J92.1, J92.10, J92.11, J92.12, J92.13, J92.14, J92.15, J92.16, J92.17, J92.18, J92.19, J92.2, J92.20, J92.3, J92.4, J92.5, J92.6, J92.7, J92.8, J92.9, JP20.1, JP21.1, JP23.1, JP24.1; no longer PAD17.P, PAD22.P, PAD23.P, PAD24.P, PAD25.P, PAD26.P, PAD27.P, PAD276.P, PAD277.P, PAD28.P, PAD285.P, PAD286.P, PAD29.P, PAD30.P, PAD31.P, PAD32.P, PAD326.P, PAD327.P, PAD328.P, PAD329.P, PAD33.P, PAD330.P, PAD331.P, PAD339.P, PAD36.P, PAD38.P, PAD4.P, PAD421.P, PAD422.P, PAD423.P, PAD424.P, PAD425.P, PAD426.P, PAD427.P, PAD428.P, PAD429.P, PAD430.P, PAD431.P, PAD432.P, PAD433.P, PAD434.P, PAD435.P, PAD436.P, PAD439.P, PAD440.P, PAD441.P
- net N$1: now also J2.1, J2.2, J2.3, J2.4, J2.5, J2.6; no longer PAD391.P, PAD392.P, PAD393.P, PAD394.P, PAD42.P, PAD43.P, PAD44.P
- net N$10: now also J11.1, J11.2, J11.3, J11.4, J11.5, J11.6; no longer PAD106.P, PAD107.P, PAD108.P, PAD109.P, PAD110.P, PAD111.P, PAD112.P
- net N$11: now also J12.1, J12.2, J12.3, J12.4, J12.5, J12.6; no longer PAD115.P, PAD116.P, PAD117.P, PAD118.P, PAD119.P, PAD120.P, PAD121.P
- net N$12: now also J13.1, J13.2, J13.3, J13.4, J13.5, J13.6; no longer PAD124.P, PAD125.P, PAD126.P, PAD127.P, PAD128.P, PAD129.P, PAD130.P
- net N$13: now also J14.1, J14.2, J14.3, J14.4, J14.5, J14.6; no longer PAD133.P, PAD134.P, PAD135.P, PAD136.P, PAD137.P, PAD138.P, PAD139.P
- net N$14: now also J15.1, J15.2, J15.3, J15.4, J15.5, J15.6; no longer PAD142.P, PAD143.P, PAD144.P, PAD145.P, PAD146.P, PAD147.P, PAD148.P
- net N$15: now also J16.1, J16.2, J16.3, J16.4, J16.5, J16.6; no longer PAD151.P, PAD152.P, PAD153.P, PAD154.P, PAD155.P, PAD156.P, PAD157.P
- net N$16: now also J17.1, J17.2, J17.3, J17.4, J17.5, J17.6; no longer PAD160.P, PAD161.P, PAD162.P, PAD163.P, PAD164.P, PAD165.P, PAD166.P
- net N$17: now also J18.1, J18.2, J18.3, J18.4, J18.5, J18.6; no longer PAD169.P, PAD170.P, PAD171.P, PAD172.P, PAD173.P, PAD174.P, PAD175.P
- net N$18: now also J19.1, J19.2, J19.3, J19.4, J19.5, J19.6; no longer PAD178.P, PAD179.P, PAD180.P, PAD181.P, PAD182.P, PAD183.P, PAD184.P
- net N$19: now also J20.1, J20.2, J20.3, J20.4, J20.5, J20.6; no longer PAD187.P, PAD188.P, PAD189.P, PAD190.P, PAD191.P, PAD192.P, PAD193.P
- net N$2: now also J3.1, J3.2, J3.3, J3.4, J3.5, J3.6; no longer PAD241.P, PAD248.P
- net N$20: now also J21.1, J21.2, J21.3, J21.4, J21.5, J21.6; no longer PAD196.P, PAD197.P, PAD198.P, PAD199.P, PAD200.P, PAD201.P, PAD202.P
- net N$21: now also J22.1, J22.2, J22.3, J22.4, J22.5, J22.6; no longer PAD205.P, PAD206.P, PAD207.P, PAD208.P, PAD209.P, PAD210.P, PAD211.P
- net N$22: now also J23.1, J23.2, J23.3, J23.4, J23.5, J23.6; no longer PAD214.P, PAD215.P, PAD216.P, PAD217.P, PAD218.P, PAD219.P, PAD220.P
- net N$23: now also J24.1, J24.2, J24.3, J24.4, J24.5, J24.6, J24.7; no longer PAD66.P, PAD67.P, PAD68.P, PAD69.P, PAD70.P, PAD71.P, PAD72.P
- net N$24: now also J25.1, J25.2, J25.3, J25.4, J25.5, J25.6, J25.7; no longer PAD73.P, PAD74.P, PAD75.P, PAD76.P, PAD77.P, PAD78.P, PAD86.P
- net N$25: now also J26.1, J26.2, J26.3, J26.4, J26.5, J26.6, J26.7; no longer PAD104.P, PAD105.P, PAD113.P, PAD114.P, PAD87.P, PAD95.P, PAD96.P
- net N$26: now also J27.1, J27.2, J27.3, J27.4, J27.5, J27.6, J27.7; no longer PAD122.P, PAD123.P, PAD131.P, PAD132.P
- net N$27: now also J28.1, J28.2, J28.3, J28.4, J28.5, J28.6, J28.7; no longer PAD260.P, PAD261.P, PAD262.P, PAD263.P, PAD264.P, PAD265.P, PAD266.P
- net N$28: now also J29.1, J29.2, J29.3, J29.4, J29.5, J29.6, J29.7; no longer PAD269.P, PAD270.P, PAD271.P, PAD272.P, PAD273.P, PAD274.P, PAD275.P
- net N$29: now also J30.1, J30.2, J30.3, J30.4, J30.5, J30.6, J30.7; no longer PAD278.P, PAD279.P, PAD280.P, PAD281.P, PAD282.P, PAD283.P, PAD284.P
- net N$3: now also J4.1, J4.2, J4.3, J4.4, J4.5, J4.6; no longer PAD1.P, PAD2.P, PAD3.P, PAD34.P, PAD35.P, PAD37.P, PAD40.P
- net N$30: now also J31.1, J31.2, J31.3, J31.4, J31.5, J31.6, J31.7; no longer PAD287.P, PAD288.P, PAD289.P, PAD290.P, PAD291.P, PAD292.P, PAD293.P
- net N$31: now also J32.1, J32.2, J32.3, J32.4, J32.5, J32.6, J32.7; no longer PAD296.P, PAD297.P, PAD298.P, PAD299.P, PAD300.P, PAD301.P, PAD302.P
- net N$32: now also J33.1, J33.2, J33.3, J33.4, J33.5, J33.6, J33.7; no longer PAD305.P, PAD306.P, PAD307.P, PAD308.P, PAD309.P, PAD310.P, PAD311.P
- net N$33: now also J34.1, J34.2, J34.3, J34.4, J34.5, J34.6, J34.7; no longer PAD314.P, PAD315.P, PAD316.P, PAD317.P, PAD318.P, PAD319.P, PAD320.P
- net N$34: now also J35.1, J35.2, J35.3, J35.4, J35.5, J35.6, J35.7; no longer PAD150.P, PAD158.P, PAD159.P, PAD167.P, PAD168.P, PAD176.P, PAD177.P
- net N$35: now also J36.1, J36.2, J36.3, J36.4, J36.5, J36.6, J36.7; no longer PAD332.P, PAD333.P, PAD334.P, PAD335.P, PAD336.P, PAD337.P, PAD338.P
- net N$36: now also J37.1, J37.2, J37.3, J37.4, J37.5, J37.6, J37.7; no longer PAD341.P, PAD342.P, PAD343.P, PAD344.P, PAD345.P, PAD346.P, PAD347.P
- net N$37: now also J38.1, J38.2, J38.3, J38.4, J38.5, J38.6, J38.7; no longer PAD350.P, PAD351.P, PAD352.P, PAD353.P, PAD354.P, PAD355.P, PAD356.P
- net N$38: now also J39.1, J39.2, J39.3, J39.4, J39.5, J39.6, J39.7; no longer PAD359.P, PAD360.P, PAD361.P, PAD362.P, PAD363.P, PAD364.P, PAD365.P
- net N$39: now also J40.1, J40.2, J40.3, J40.4, J40.5, J40.6, J40.7; no longer PAD368.P, PAD369.P, PAD370.P, PAD371.P, PAD372.P, PAD373.P, PAD374.P
- net N$4: now also J5.1, J5.2, J5.3, J5.4, J5.5, J5.6; no longer PAD45.P, PAD46.P, PAD47.P, PAD48.P, PAD49.P, PAD50.P, PAD51.P
- net N$40: now also J41.1, J41.2, J41.3, J41.4, J41.5, J41.6, J41.7; no longer PAD377.P, PAD378.P, PAD379.P, PAD380.P, PAD381.P, PAD382.P, PAD383.P
- net N$41: now also J42.1, J42.2, J42.3, J42.4, J42.5, J42.6, J42.7; no longer PAD385.P, PAD386.P, PAD387.P, PAD388.P, PAD389.P, PAD39.P, PAD41.P
- net N$42: now also J43.1, J43.2, J43.3, J43.4, J43.5, J43.6, J43.7; no longer PAD242.P, PAD247.P
- net N$43: now also J44.1, J44.2, J44.3, J44.4, J44.5, J44.6, J44.7; no longer PAD243.P, PAD246.P
- net N$44: now also J45.1, J45.2, J45.3, J45.4, J45.5, J45.6, J45.7; no longer PAD244.P, PAD245.P
- net N$45: now also J46.1, J46.2, J46.3, J46.4, J46.5, J46.6, J46.7; no longer PAD185.P, PAD186.P, PAD194.P, PAD195.P, PAD203.P, PAD204.P, PAD212.P
- net N$46: now also J47.1, J47.2, J47.3, J47.4, J47.5, J47.6, J47.7; no longer PAD249.P, PAD250.P, PAD251.P, PAD252.P, PAD253.P, PAD254.P, PAD255.P
- net N$49: now also J50.1, J50.2, J50.3, J50.4, J50.5, J50.6, J50.7; no longer PAD213.P, PAD221.P, PAD222.P, PAD223.P, PAD224.P, PAD225.P, PAD226.P
- net N$5: now also J6.1, J6.2, J6.3, J6.4, J6.5, J6.6; no longer PAD52.P, PAD53.P, PAD54.P, PAD55.P, PAD56.P, PAD57.P, PAD58.P
- net N$50: now also J51.1, J51.2, J51.3, J51.4, J51.5, J51.6, J51.7; no longer PAD227.P, PAD228.P, PAD229.P, PAD230.P, PAD231.P, PAD232.P, PAD233.P
- net N$51: now also J52.1, J52.2, J52.3, J52.4, J52.5, J52.6, J52.7; no longer PAD234.P, PAD235.P, PAD236.P, PAD237.P, PAD238.P, PAD239.P, PAD240.P
- net N$59: now also J60.1, J60.2, J60.3, J60.4, J60.5, J60.6, J60.7; no longer PAD340.P, PAD348.P, PAD349.P, PAD357.P, PAD358.P, PAD366.P, PAD367.P
- net N$6: now also J7.1, J7.2, J7.3, J7.4, J7.5, J7.6; no longer PAD59.P, PAD60.P, PAD61.P, PAD62.P, PAD63.P, PAD64.P, PAD65.P
- net N$60: now also J61.1, J61.2, J61.3, J61.4, J61.5, J61.6, J61.7; no longer PAD375.P, PAD376.P, PAD384.P, PAD390.P, PAD395.P, PAD414.P, PAD415.P
- net N$61: now also J62.1, J62.2, J62.3, J62.4, J62.5, J62.6, J62.7; no longer PAD416.P, PAD420.P, PAD437.P, PAD438.P, PAD457.P, PAD458.P, PAD463.P
- net N$62: now also J63.1, J63.2, J63.3, J63.4, J63.5, J63.6, J63.7; no longer PAD464.P, PAD465.P, PAD466.P, PAD467.P, PAD468.P, PAD469.P, PAD470.P
- net N$63: now also J64.1, J64.2, J64.3, J64.4, J64.5, J64.6, J64.7; no longer PAD140.P, PAD141.P, PAD149.P, PAD471.P, PAD472.P, PAD473.P, PAD474.P
- net N$64: now also J65.1, J65.2, J65.3, J65.4, J65.5, J65.6, J65.7; no longer PAD475.P, PAD476.P, PAD477.P, PAD478.P, PAD479.P, PAD480.P, PAD481.P
- net N$65: now also J66.1, J66.2, J66.3, J66.4, J66.5, J66.6, J66.7; no longer PAD482.P, PAD483.P, PAD484.P, PAD485.P, PAD486.P, PAD487.P, PAD488.P
- net N$66: now also J67.1, J67.2, J67.3, J67.4, J67.5, J67.6, J67.7; no longer PAD489.P, PAD490.P, PAD491.P, PAD492.P, PAD493.P, PAD494.P, PAD495.P
- net N$67: now also J68.1, J68.2, J68.3, J68.4, J68.5, J68.6, J68.7; no longer PAD496.P, PAD497.P, PAD498.P, PAD499.P, PAD500.P, PAD501.P, PAD502.P
- net N$68: now also J69.1, J69.2, J69.3, J69.4, J69.5, J69.6, J69.7; no longer PAD503.P, PAD504.P, PAD505.P, PAD506.P, PAD507.P, PAD508.P, PAD509.P
- net N$69: now also J70.1, J70.2, J70.3, J70.4, J70.5, J70.6, J70.7; no longer PAD510.P, PAD511.P, PAD512.P, PAD513.P, PAD514.P, PAD515.P, PAD516.P
- net N$7: now also J8.1, J8.2, J8.3, J8.4, J8.5, J8.6; no longer PAD79.P, PAD80.P, PAD81.P, PAD82.P, PAD83.P, PAD84.P, PAD85.P
- net N$70: now also J71.1, J71.2, J71.3, J71.4, J71.5, J71.6, J71.7; no longer PAD517.P, PAD518.P, PAD519.P, PAD520.P, PAD521.P, PAD522.P, PAD523.P
- net N$71: now also J72.1, J72.2, J72.3, J72.4, J72.5, J72.6, J72.7; no longer PAD524.P, PAD525.P, PAD526.P, PAD527.P, PAD528.P, PAD529.P, PAD530.P
- net N$72: now also J73.1, J73.2, J73.3, J73.4, J73.5, J73.6, J73.7; no longer PAD531.P, PAD532.P, PAD533.P, PAD534.P, PAD535.P, PAD536.P, PAD537.P
- net N$73: now also J74.1, J74.2, J74.3, J74.4, J74.5, J74.6, J74.7; no longer PAD538.P, PAD539.P, PAD540.P, PAD541.P, PAD542.P, PAD543.P, PAD544.P
- net N$74: now also J75.1, J75.2, J75.3, J75.4, J75.5, J75.6, J75.7; no longer PAD545.P, PAD546.P, PAD547.P, PAD548.P, PAD549.P, PAD550.P, PAD551.P
- net N$75: now also J76.1, J76.2, J76.3, J76.4, J76.5, J76.6, J76.7; no longer PAD552.P, PAD553.P, PAD554.P, PAD555.P, PAD556.P, PAD557.P, PAD558.P
- net N$76: now also J77.1, J77.2, J77.3, J77.4, J77.5, J77.6, J77.7; no longer PAD559.P, PAD560.P, PAD561.P, PAD562.P, PAD563.P, PAD564.P, PAD565.P
- net N$77: now also J78.1, J78.2, J78.3, J78.4, J78.5, J78.6, J78.7; no longer PAD566.P, PAD567.P, PAD568.P, PAD569.P, PAD570.P, PAD571.P, PAD572.P
- net N$78: now also J79.1, J79.2, J79.3, J79.4, J79.5, J79.6, J79.7; no longer PAD573.P, PAD574.P, PAD575.P, PAD576.P, PAD577.P, PAD578.P, PAD579.P
- net N$79: now also J80.1, J80.2, J80.3, J80.4, J80.5, J80.6, J80.7; no longer PAD580.P, PAD581.P, PAD582.P, PAD583.P, PAD584.P, PAD585.P, PAD586.P
- net N$8: now also J9.1, J9.2, J9.3, J9.4, J9.5, J9.6; no longer PAD88.P, PAD89.P, PAD90.P, PAD91.P, PAD92.P, PAD93.P, PAD94.P
- net N$80: now also J81.1, J81.2, J81.3, J81.4, J81.5, J81.6, J81.7; no longer PAD587.P, PAD588.P, PAD589.P, PAD590.P, PAD591.P, PAD592.P, PAD593.P
- net N$81: now also J82.1, J82.2, J82.3, J82.4, J82.5, J82.6, J82.7; no longer PAD594.P, PAD595.P, PAD596.P, PAD597.P, PAD598.P, PAD599.P, PAD600.P
- net N$82: now also J83.1, J83.2, J83.3, J83.4, J83.5, J83.6, J83.7; no longer PAD601.P, PAD602.P, PAD603.P, PAD604.P, PAD605.P, PAD606.P, PAD607.P
- net N$83: now also J84.1, J84.2, J84.3, J84.4, J84.5, J84.6, J84.7; no longer PAD608.P, PAD609.P, PAD610.P, PAD611.P, PAD612.P, PAD613.P, PAD614.P
- net N$84: now also J85.1, J85.2, J85.3, J85.4, J85.5, J85.6, J85.7; no longer PAD615.P, PAD616.P, PAD617.P, PAD618.P, PAD619.P, PAD620.P, PAD621.P
- net N$9: now also J10.1, J10.2, J10.3, J10.4, J10.5, J10.6; no longer PAD100.P, PAD101.P, PAD102.P, PAD103.P, PAD97.P, PAD98.P, PAD99.P
- net N$92: now also JP13.1, JP5.1; no longer PAD643.P, PAD644.P, PAD645.P, PAD646.P, PAD647.P, PAD648.P, PAD649.P
- net N$93: now also JP14.1, JP6.1; no longer PAD650.P, PAD651.P, PAD652.P, PAD653.P, PAD654.P, PAD655.P, PAD656.P
- net N$94: now also JP15.1, JP7.1; no longer PAD657.P, PAD658.P, PAD659.P, PAD660.P, PAD661.P, PAD662.P, PAD663.P
- net N$95: now also JP16.1, JP8.1; no longer PAD664.P, PAD665.P, PAD666.P, PAD667.P, PAD668.P, PAD669.P, PAD670.P
- net N$96: now also JP17.1, JP9.1; no longer PAD671.P, PAD672.P, PAD673.P, PAD674.P, PAD675.P, PAD676.P, PAD677.P
- net VDD: now also J90.1, J90.10, J90.11, J90.12, J90.13, J90.14, J90.15, J90.16, J90.17, J90.18, J90.19, J90.2, J90.20, J90.3, J90.4, J90.5, J90.6, J90.7, J90.8, J90.9, J93.1, J93.10, J93.11, J93.12, J93.13, J93.14, J93.15, J93.16, J93.17, J93.18, J93.19, J93.2, J93.20, J93.3, J93.4, J93.5, J93.6, J93.7, J93.8, J93.9, JP18.1, JP19.1, JP22.1, JP25.1; no longer PAD10.P, PAD11.P, PAD12.P, PAD13.P, PAD14.P, PAD15.P, PAD16.P, PAD18.P, PAD19.P, PAD20.P, PAD21.P, PAD294.P, PAD295.P, PAD303.P, PAD304.P, PAD312.P, PAD313.P, PAD321.P, PAD322.P, PAD323.P, PAD324.P, PAD325.P, PAD442.P, PAD443.P, PAD444.P, PAD445.P, PAD446.P, PAD447.P, PAD448.P, PAD449.P, PAD450.P, PAD451.P, PAD452.P, PAD453.P, PAD454.P, PAD455.P, PAD456.P, PAD459.P, PAD460.P, PAD461.P, PAD462.P, PAD5.P, PAD6.P, PAD7.P, PAD8.P, PAD9.P

Commit message: Change usb connector
Change to correct usb connecter and moved esp8266 bit more onto the
board.
Parts:
- removed JP1: USB-RECEPTABLE, daspilker:USB-RECEPTABLE
- added X1: (no value), microbuilder:USBMICRO_20329
Connections:
- net GND: now also X1.GND; no longer JP1.GND
- net VCC: now also X1.VBUS; no longer JP1.VCC
Changed lines of the file:
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@@
 <part name="VDD1" library="supply1" deviceset="VDD" device=""/>
 <part name="U1" library="SparkFun-PowerIC" deviceset="V_REG_MIC5205" device="3.3V" value="3.3V/150mA"/>
-<part name="JP1" library="daspilker" deviceset="USB-RECEPTABLE" device=""/>
 <part name="SUPPLY1" library="supply2" deviceset="VCC" device=""/>
 <part name="GND5" library="supply1" deviceset="GND" device=""/>
 <part name="VDD4" library="supply1" deviceset="VDD" device=""/>
-<part name="SUPPLY2" library="supply2" deviceset="VCC" device=""/>
-<part name="GND6" library="supply1" deviceset="GND" device=""/>
 <part name="J24" library="SparkFun-Connectors" deviceset="M07" device="NO_SILK"/>
 <part name="J25" library="SparkFun-Connectors" deviceset="M07" device="NO_SILK"/>
@@
 <part name="JP24" library="adafruit" deviceset="PINHD-1X1" device="CB"/>
 <part name="JP25" library="adafruit" deviceset="PINHD-1X1" device="CB"/>
+<part name="X1" library="microbuilder" deviceset="USB" device="MICRO_20329"/>
+<part name="SUPPLY5" library="supply2" deviceset="VCC" device=""/>
+<part name="GND2" library="supply1" deviceset="GND" device=""/>
 </parts>
 <sheets>
@@
 <instance part="VDD1" gate="G$1" x="-7.62" y="71.12"/>
 <instance part="U1" gate="U1" x="-25.4" y="88.9"/>
-<instance part="JP1" gate="G$1" x="-40.64" y="30.48"/>
 <instance part="SUPPLY1" gate="G$1" x="-43.18" y="99.06"/>
 <instance part="GND5" gate="1" x="-43.18" y="78.74"/>
 <instance part="VDD4" gate="G$1" x="-10.16" y="99.06"/>
-<instance part="SUPPLY2" gate="G$1" x="-53.34" y="40.64"/>
-<instance part="GND6" gate="1" x="-53.34" y="17.78"/>
 <instance part="J24" gate="G$1" x="86.36" y="63.5"/>
 <instance part="J25" gate="G$1" x="99.06" y="63.5"/>
@@
 <instance part="JP24" gate="G$1" x="-12.7" y="-73.66" rot="R180"/>
 <instance part="JP25" gate="G$1" x="-55.88" y="-76.2" rot="R180"/>
+<instance part="X1" gate="G$1" x="-78.74" y="27.94"/>
+<instance part="SUPPLY5" gate="G$1" x="-66.04" y="40.64"/>
+<instance part="GND2" gate="1" x="-66.04" y="15.24"/>
 </instances>
 <busses>
@@
 <pinref part="DC" gate="G$1" pin="GND"/>
 <wire x1="-27.94" y1="50.8" x2="-27.94" y2="55.88" width="0.1524" layer="91"/>
-</segment>
-<segment>
-<pinref part="JP1" gate="G$1" pin="GND"/>
-<pinref part="GND6" gate="1" pin="GND"/>
-<wire x1="-48.26" y1="25.4" x2="-53.34" y2="25.4" width="0.1524" layer="91"/>
-<wire x1="-53.34" y1="25.4" x2="-53.34" y2="20.32" width="0.1524" layer="91"/>
 </segment>
 <segment>
@@
 <wire x1="-5.08" y1="-78.74" x2="-5.08" y2="-83.82" width="0.1524" layer="91"/>
 </segment>
+<segment>
+<pinref part="X1" gate="G$1" pin="GND"/>
+<pinref part="GND2" gate="1" pin="GND"/>
+<wire x1="-68.58" y1="22.86" x2="-66.04" y2="22.86" width="0.1524" layer="91"/>
+<wire x1="-66.04" y1="22.86" x2="-66.04" y2="17.78" width="0.1524" layer="91"/>
+</segment>
 </net>
 <net name="VCC" class="0">
@@
 <pinref part="DC" gate="G$1" pin="VIN"/>
 <wire x1="-45.72" y1="63.5" x2="-40.64" y2="63.5" width="0.1524" layer="91"/>
-</segment>
-<segment>
-<pinref part="JP1" gate="G$1" pin="VCC"/>
-<pinref part="SUPPLY2" gate="G$1" pin="VCC"/>
-<wire x1="-48.26" y1="35.56" x2="-53.34" y2="35.56" width="0.1524" layer="91"/>
-<wire x1="-53.34" y1="35.56" x2="-53.34" y2="38.1" width="0.1524" layer="91"/>
 </segment>
 <segment>
@@
 <junction x="-43.18" y="93.98"/>
 </segment>
+<segment>
+<pinref part="X1" gate="G$1" pin="VBUS"/>
+<pinref part="SUPPLY5" gate="G$1" pin="VCC"/>
+<wire x1="-68.58" y1="33.02" x2="-66.04" y2="33.02" width="0.1524" layer="91"/>
+<wire x1="-66.04" y1="33.02" x2="-66.04" y2="38.1" width="0.1524" layer="91"/>
+</segment>
 </net>
