File: MX2-8-7/Protoboard MX2-8-7.sch (EAGLE design)
At the start: 140 parts, among them J1 DCJ0202

Commit message: Change usb connector
Change to correct usb connecter and moved esp8266 bit more onto the
board.
Parts:
- removed JP11: (no value), adafruit:PINHD-1X1CB
- removed JP17: (no value), adafruit:PINHD-1X1-BIGPOGO
Connections:
- removed net N$45: JP11.1, JP17.1
Changed lines of the file:
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@@
 <part name="JP9" library="adafruit" deviceset="PINHD-1X1" device="CB"/>
 <part name="JP10" library="adafruit" deviceset="PINHD-1X1" device="CB"/>
-<part name="JP11" library="adafruit" deviceset="PINHD-1X1" device="CB"/>
 <part name="JP12" library="adafruit" deviceset="PINHD-1X1" device="-BIGPOGO"/>
 <part name="JP13" library="adafruit" deviceset="PINHD-1X1" device="-BIGPOGO"/>
@@
 <part name="JP15" library="adafruit" deviceset="PINHD-1X1" device="-BIGPOGO"/>
 <part name="JP16" library="adafruit" deviceset="PINHD-1X1" device="-BIGPOGO"/>
-<part name="JP17" library="adafruit" deviceset="PINHD-1X1" device="-BIGPOGO"/>
 </parts>
 <sheets>
@@
 <instance part="JP9" gate="G$1" x="162.56" y="-27.94"/>
 <instance part="JP10" gate="G$1" x="172.72" y="-27.94"/>
-<instance part="JP11" gate="G$1" x="182.88" y="-27.94"/>
 <instance part="JP12" gate="G$1" x="129.54" y="-38.1" rot="R270"/>
 <instance part="JP13" gate="G$1" x="139.7" y="-38.1" rot="R270"/>
@@
 <instance part="JP15" gate="G$1" x="160.02" y="-38.1" rot="R270"/>
 <instance part="JP16" gate="G$1" x="170.18" y="-38.1" rot="R270"/>
-<instance part="JP17" gate="G$1" x="180.34" y="-38.1" rot="R270"/>
 </instances>
 <busses>
@@
 </segment>
 </net>
-<net name="N$45" class="0">
-<segment>
-<pinref part="JP17" gate="G$1" pin="1"/>
-<pinref part="JP11" gate="G$1" pin="1"/>
-<wire x1="180.34" y1="-35.56" x2="180.34" y2="-27.94" width="0.1524" layer="91"/>
-</segment>
-</net>

Commit message: Update esp component and usb
test
Parts:
- removed JP2, JP5, JP6: (no value), adafruit:PINHD-1X3CB
- removed JP3, JP4: (no value), adafruit:PINHD-1X1CB
- added J39: (no value), SparkFun-Connectors:M06NO_SILK_FEMALE_PTH
- added J40: (no value), SparkFun-Connectors:M05NO_SILK
- added U1: (no value), SparkFun-PowerIC:MIC52053.3V
- added X1: (no value), microbuilder:USB_MICRO_20329_V2
Connections:
- net GND: now also U1.GND, X1.GND
- net N$40: now also J39.1, J39.2, J39.3, J39.4, J39.5, J39.6; no longer JP5.1, JP5.2, JP5.3, JP6.1, JP6.2, JP6.3
- net N$41: now also J40.1, J40.2, J40.3, J40.4, J40.5; no longer JP2.1, JP2.2, JP2.3, JP3.1, JP4.1
- net VCC: now also U1.EN, U1.IN, X1.VBUS
- net VDD: now also U1.OUT
Changed lines of the file:
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@@
 <part name="J37" library="SparkFun-Connectors" deviceset="M09" device="NO_SILK"/>
 <part name="J38" library="SparkFun-Connectors" deviceset="M09" device="NO_SILK"/>
-<part name="JP2" library="adafruit" deviceset="PINHD-1X3" device="CB"/>
-<part name="JP3" library="adafruit" deviceset="PINHD-1X1" device="CB"/>
-<part name="JP4" library="adafruit" deviceset="PINHD-1X1" device="CB"/>
-<part name="JP5" library="adafruit" deviceset="PINHD-1X3" device="CB"/>
-<part name="JP6" library="adafruit" deviceset="PINHD-1X3" device="CB"/>
 <part name="JP1" library="adafruit" deviceset="PINHD-1X1" device="CB"/>
 <part name="JP7" library="adafruit" deviceset="PINHD-1X1" device="CB"/>
@@
 <part name="JP15" library="adafruit" deviceset="PINHD-1X1" device="-BIGPOGO"/>
 <part name="JP16" library="adafruit" deviceset="PINHD-1X1" device="-BIGPOGO"/>
+<part name="U1" library="SparkFun-PowerIC" deviceset="MIC5205" device="3.3V"/>
+<part name="VDD4" library="supply1" deviceset="VDD" device=""/>
+<part name="SUPPLY1" library="supply2" deviceset="VCC" device=""/>
+<part name="GND5" library="supply1" deviceset="GND" device=""/>
+<part name="J39" library="SparkFun-Connectors" deviceset="M06" device="NO_SILK_FEMALE_PTH"/>
+<part name="J40" library="SparkFun-Connectors" deviceset="M05" device="NO_SILK"/>
+<part name="X1" library="microbuilder" deviceset="USB" device="_MICRO_20329_V2"/>
+<part name="SUPPLY2" library="supply2" deviceset="VCC" device=""/>
+<part name="GND6" library="supply1" deviceset="GND" device=""/>
 </parts>
 <sheets>
@@
 <instance part="J37" gate="G$1" x="271.78" y="5.08"/>
 <instance part="J38" gate="G$1" x="284.48" y="5.08"/>
-<instance part="JP2" gate="A" x="322.58" y="10.16"/>
-<instance part="JP3" gate="G$1" x="322.58" y="0"/>
-<instance part="JP4" gate="G$1" x="322.58" y="-7.62"/>
-<instance part="JP5" gate="A" x="307.34" y="12.7"/>
-<instance part="JP6" gate="A" x="307.34" y="2.54"/>
 <instance part="JP1" gate="G$1" x="132.08" y="-27.94"/>
 <instance part="JP7" gate="G$1" x="142.24" y="-27.94"/>
@@
 <instance part="JP15" gate="G$1" x="160.02" y="-38.1" rot="R270"/>
 <instance part="JP16" gate="G$1" x="170.18" y="-38.1" rot="R270"/>
+<instance part="U1" gate="G$1" x="-40.64" y="27.94"/>
+<instance part="VDD4" gate="G$1" x="-33.02" y="40.64"/>
+<instance part="SUPPLY1" gate="G$1" x="-53.34" y="40.64"/>
+<instance part="GND5" gate="1" x="-53.34" y="15.24"/>
+<instance part="J39" gate="G$1" x="304.8" y="7.62"/>
+<instance part="J40" gate="G$1" x="320.04" y="10.16"/>
+<instance part="X1" gate="G$1" x="-45.72" y="-12.7"/>
+<instance part="SUPPLY2" gate="G$1" x="-33.02" y="-2.54"/>
+<instance part="GND6" gate="1" x="-33.02" y="-25.4"/>
 </instances>
 <busses>
@@
 <wire x1="-27.94" y1="50.8" x2="-27.94" y2="55.88" width="0.1524" layer="91"/>
 </segment>
+<segment>
+<pinref part="U1" gate="G$1" pin="GND"/>
+<pinref part="GND5" gate="1" pin="GND"/>
+<wire x1="-50.8" y1="22.86" x2="-53.34" y2="22.86" width="0.1524" layer="91"/>
+<wire x1="-53.34" y1="22.86" x2="-53.34" y2="17.78" width="0.1524" layer="91"/>
+</segment>
+<segment>
+<pinref part="X1" gate="G$1" pin="GND"/>
+<pinref part="GND6" gate="1" pin="GND"/>
+<wire x1="-35.56" y1="-17.78" x2="-33.02" y2="-17.78" width="0.1524" layer="91"/>
+<wire x1="-33.02" y1="-17.78" x2="-33.02" y2="-22.86" width="0.1524" layer="91"/>
+</segment>
 </net>
 <net name="VCC" class="0">
@@
 <pinref part="DC" gate="G$1" pin="VIN"/>
 <wire x1="-45.72" y1="63.5" x2="-40.64" y2="63.5" width="0.1524" layer="91"/>
+</segment>
+<segment>
+<pinref part="U1" gate="G$1" pin="IN"/>
+<pinref part="SUPPLY1" gate="G$1" pin="VCC"/>
+<wire x1="-50.8" y1="33.02" x2="-53.34" y2="33.02" width="0.1524" layer="91"/>
+<wire x1="-53.34" y1="33.02" x2="-53.34" y2="38.1" width="0.1524" layer="91"/>
+<pinref part="U1" gate="G$1" pin="EN"/>
+<wire x1="-50.8" y1="27.94" x2="-53.34" y2="27.94" width="0.1524" layer="91"/>
+<wire x1="-53.34" y1="27.94" x2="-53.34" y2="33.02" width="0.1524" layer="91"/>
+<junction x="-53.34" y="33.02"/>
+</segment>
+<segment>
+<pinref part="X1" gate="G$1" pin="VBUS"/>
+<pinref part="SUPPLY2" gate="G$1" pin="VCC"/>
+<wire x1="-35.56" y1="-7.62" x2="-33.02" y2="-7.62" width="0.1524" layer="91"/>
+<wire x1="-33.02" y1="-7.62" x2="-33.02" y2="-5.08" width="0.1524" layer="91"/>
 </segment>
 </net>
@@
 <wire x1="-7.62" y1="63.5" x2="-7.62" y2="68.58" width="0.1524" layer="91"/>
 </segment>
+<segment>
+<pinref part="U1" gate="G$1" pin="OUT"/>
+<pinref part="VDD4" gate="G$1" pin="VDD"/>
+<wire x1="-33.02" y1="33.02" x2="-33.02" y2="38.1" width="0.1524" layer="91"/>
+</segment>
 </net>
 <net name="N$1" class="0">
@@
 </segment>
 </net>
-<net name="N$41" class="0">
-<segment>
-<pinref part="JP4" gate="G$1" pin="1"/>
-<pinref part="JP3" gate="G$1" pin="1"/>
-<wire x1="320.04" y1="-7.62" x2="320.04" y2="0" width="0.1524" layer="91"/>
-<pinref part="JP2" gate="A" pin="3"/>
-<wire x1="320.04" y1="0" x2="320.04" y2="7.62" width="0.1524" layer="91"/>
-<pinref part="JP2" gate="A" pin="2"/>
-<wire x1="320.04" y1="7.62" x2="320.04" y2="10.16" width="0.1524" layer="91"/>
-<pinref part="JP2" gate="A" pin="1"/>
-<wire x1="320.04" y1="10.16" x2="320.04" y2="12.7" width="0.1524" layer="91"/>
-</segment>
-</net>
-<net name="N$40" class="0">
-<segment>
-<pinref part="JP5" gate="A" pin="1"/>
-<pinref part="JP5" gate="A" pin="2"/>
-<wire x1="304.8" y1="15.24" x2="304.8" y2="12.7" width="0.1524" layer="91"/>
-<pinref part="JP5" gate="A" pin="3"/>
-<wire x1="304.8" y1="12.7" x2="304.8" y2="10.16" width="0.1524" layer="91"/>
-<pinref part="JP6" gate="A" pin="1"/>
-<wire x1="304.8" y1="10.16" x2="304.8" y2="5.08" width="0.1524" layer="91"/>
-<pinref part="JP6" gate="A" pin="2"/>
-<wire x1="304.8" y1="5.08" x2="304.8" y2="2.54" width="0.1524" layer="91"/>
-<pinref part="JP6" gate="A" pin="3"/>
-<wire x1="304.8" y1="2.54" x2="304.8" y2="0" width="0.1524" layer="91"/>
-</segment>
-</net>
 <net name="N$2" class="0">
 <segment>
@@
 </segment>
 </net>
+<net name="N$40" class="0">
+<segment>
+<pinref part="J39" gate="G$1" pin="1"/>
+<pinref part="J39" gate="G$1" pin="2"/>
+<wire x1="309.88" y1="2.54" x2="309.88" y2="5.08" width="0.1524" layer="91"/>
+<pinref part="J39" gate="G$1" pin="3"/>
+<wire x1="309.88" y1="5.08" x2="309.88" y2="7.62" width="0.1524" layer="91"/>
+<pinref part="J39" gate="G$1" pin="4"/>
+<wire x1="309.88" y1="7.62" x2="309.88" y2="10.16" width="0.1524" layer="91"/>
+<pinref part="J39" gate="G$1" pin="5"/>
+<wire x1="309.88" y1="10.16" x2="309.88" y2="12.7" width="0.1524" layer="91"/>
+<pinref part="J39" gate="G$1" pin="6"/>
+<wire x1="309.88" y1="12.7" x2="309.88" y2="15.24" width="0.1524" layer="91"/>
+</segment>
+</net>
+<net name="N$41" class="0">
+<segment>
+<pinref part="J40" gate="G$1" pin="1"/>
+<pinref part="J40" gate="G$1" pin="2"/>
+<wire x1="327.66" y1="5.08" x2="327.66" y2="7.62" width="0.1524" layer="91"/>
+<pinref part="J40" gate="G$1" pin="3"/>
+<wire x1="327.66" y1="7.62" x2="327.66" y2="10.16" width="0.1524" layer="91"/>
+<pinref part="J40" gate="G$1" pin="4"/>
+<wire x1="327.66" y1="10.16" x2="327.66" y2="12.7" width="0.1524" layer="91"/>
+<pinref part="J40" gate="G$1" pin="5"/>
+<wire x1="327.66" y1="12.7" x2="327.66" y2="15.24" width="0.1524" layer="91"/>
+</segment>
+</net>
