File: MX2-8-7/Protoboard MX2-8-7.brd (EAGLE design)
At the start: 64.4 x 71.2 mm, 137 parts, among them J1 DCJ0202

Commit message: Silkscreen text fixes
Silkscreen text fixes
Other:
- board text added: "MX 2-8-7 rev 2"
- board text removed: "MX 2-8-7 rev2"
Changed lines of the file:
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@@
 <wire x1="46.99" y1="19.685" x2="46.99" y2="34.925" width="0.4064" layer="25"/>
 <wire x1="49.53" y1="34.925" x2="49.53" y2="22.225" width="0.4064" layer="25"/>
-<text x="45.72" y="69.215" size="1.778" layer="25">xnsense.no</text>
-<text x="3.195" y="25.745" size="1.778" layer="25" rot="R90">MX 2-8-7 rev2</text>
+<text x="24.13" y="68.58" size="1.778" layer="25">xnsense.no</text>
+<text x="22.245" y="1.615" size="1.778" layer="25">MX 2-8-7 rev 2</text>
 <wire x1="63.9" y1="62.23" x2="54.61" y2="62.23" width="0.4064" layer="25"/>
 <wire x1="54.61" y1="62.23" x2="54.61" y2="60.325" width="0.4064" layer="25"/>
 <wire x1="63.9" y1="62.23" x2="63.9" y2="36.83" width="0.4064" layer="25"/>
-<text x="58.42" y="66.675" size="1.016" layer="25">GND</text>
-<text x="58.5" y="5.005" size="1.016" layer="25">GND</text>
+<text x="58.3" y="66.675" size="1.016" layer="25">GND</text>
+<text x="58.3" y="5.005" size="1.016" layer="25">GND</text>
 <text x="58.3" y="63.465" size="1.016" layer="25">3.3V</text>
 <text x="58.3" y="7.585" size="1.016" layer="25">3.3V</text>
