File: MX4-7-9/Protoboard MX4-7-9-ESP12.brd (EAGLE design)
At the start: 52.8 x 59.6 mm, 52 parts

Commit message: Update esp component and usb
test
Parts:
- removed MDL1: (no value), ESP8266-ESP12E:ESP8266-ESP12E
- added X1: ESP-12E, microbuilder:ESP-12E
- moved 5V 6.35 mm to (44.5, 24.8)
- moved JP1 1.91 mm to (49.2, 50.2)
- moved JP10 1.91 mm to (44.5, 41.9)
- moved JP11 1.91 mm to (44.5, 39.4)
- moved JP2 1.91 mm to (49.2, 45.1)
- moved JP7 1.91 mm to (49.2, 34.9)
- moved JP8 1.91 mm to (44.5, 47.0)
- moved JP6 1.90 mm to (49.2, 40.0)
- moved JP9 1.90 mm to (44.5, 44.5)
Connections:
- net GND: now also X1.9; no longer MDL1.9
- net N$10: now also X1.13; no longer MDL1.13
- net N$11: now also X1.12; no longer MDL1.12
- net N$12: now also X1.11; no longer MDL1.11
- net N$13: now also X1.10; no longer MDL1.10
- net N$26: now also X1.4; no longer MDL1.5
- net N$34: now also X1.7
- net N$50: now also X1.1; no longer MDL1.1
- net N$51: now also X1.2; no longer MDL1.2
- net N$52: now also X1.3; no longer MDL1.3
- net N$55: now also X1.5; no longer MDL1.6
- net N$56: now also X1.6; no longer MDL1.7
- net N$9: now also X1.14; no longer MDL1.14
- net RX: now also X1.15; no longer MDL1.15
- net TX: now also X1.16; no longer MDL1.16
- net VDD: now also X1.8; no longer MDL1.8
