File: MX4-7-9/MX4-7-9.sch (EAGLE design)
At the start: 115 parts, among them J1 DCJ0202

Commit message: Routing and Gerber files
Routed and produced gerber files
Parts:
- removed JP10, JP11, JP12, JP13, JP14, JP15, JP16, JP17, JP18, JP19, JP2, JP20, JP21, JP22, JP23, JP24, JP25, JP26, JP27, JP28, JP29, JP3, JP30, JP31, JP32, JP33, JP4, JP47, JP5, JP6, JP64, JP65, JP66, JP67, JP68, JP69, JP7, JP70, JP71, JP72, JP73, JP74, JP75, JP76, JP77, JP78, JP79, JP8, JP80, JP81, JP82, JP83, JP9: (no value), adafruit:PINHD-1X6CB
- removed JP100, JP101, JP102, JP103, JP104, JP105, JP106, JP107, JP108, JP109, JP34, JP35, JP36, JP37, JP38, JP39, JP40, JP41, JP42, JP43, JP44, JP45, JP46, JP48, JP49, JP50, JP51, JP52, JP53, JP54, JP55, JP56, JP57, JP58, JP59, JP60, JP61, JP62, JP63, JP85, JP86, JP87, JP88, JP89, JP90, JP91, JP92, JP93, JP96, JP97, JP98, JP99: (no value), adafruit:PINHD-1X1CB
- added J10, J11, J12, J13, J14, J15, J16, J17, J18, J19, J20, J21, J22, J23, J24, J25, J26, J27, J28, J29, J30, J31, J32, J33, J34, J35, J36, J37, J38, J39, J40, J41, J42, J43, J44, J45, J46, J47, J48, J49, J50, J51, J52, J53, J54, J55, J56, J57, J58, J59, J8, J9: (no value), SparkFun-Connectors:M07NO_SILK
- added J60: (no value), SparkFun-Connectors:M06NO_SILK_FEMALE_PTH
Connections:
- removed net N$57: JP81.1, JP81.2, JP81.3, JP81.4, JP81.5, JP81.6, JP92.1
- removed net N$58: JP82.1, JP82.2, JP82.3, JP82.4, JP82.5, JP82.6, JP93.1
- removed net N$59: JP83.1, JP83.2, JP83.3, JP83.4, JP83.5, JP83.6
- new net N$40: J46.1, J46.2, J46.3, J46.4, J46.5, J46.6, J46.7
- new net N$43: J48.1, J48.2, J48.3, J48.4, J48.5, J48.6, J48.7
- new net N$44: J49.1, J49.2, J49.3, J49.4, J49.5, J49.6, J49.7
- net N$1: now also J8.1, J8.2, J8.3, J8.4, J8.5, J8.6, J8.7; no longer JP2.1, JP2.2, JP2.3, JP2.4, JP2.5, JP2.6, JP48.1
- net N$10: now also J17.1, J17.2, J17.3, J17.4, J17.5, J17.6, J17.7; no longer JP54.1, JP9.1, JP9.2, JP9.3, JP9.4, JP9.5, JP9.6
- net N$11: now also J18.1, J18.2, J18.3, J18.4, J18.5, J18.6, J18.7; no longer JP10.1, JP10.2, JP10.3, JP10.4, JP10.5, JP10.6, JP55.1
- net N$12: now also J19.1, J19.2, J19.3, J19.4, J19.5, J19.6, J19.7; no longer JP11.1, JP11.2, JP11.3, JP11.4, JP11.5, JP11.6, JP56.1
- net N$13: now also J20.1, J20.2, J20.3, J20.4, J20.5, J20.6, J20.7; no longer JP12.1, JP12.2, JP12.3, JP12.4, JP12.5, JP12.6, JP57.1
- net N$14: now also J21.1, J21.2, J21.3, J21.4, J21.5, J21.6, J21.7; no longer JP13.1, JP13.2, JP13.3, JP13.4, JP13.5, JP13.6, JP58.1
- net N$15: now also J22.1, J22.2, J22.3, J22.4, J22.5, J22.6, J22.7; no longer JP14.1, JP14.2, JP14.3, JP14.4, JP14.5, JP14.6, JP59.1
- net N$16: now also J23.1, J23.2, J23.3, J23.4, J23.5, J23.6, J23.7; no longer JP15.1, JP15.2, JP15.3, JP15.4, JP15.5, JP15.6, JP60.1
- net N$17: now also J24.1, J24.2, J24.3, J24.4, J24.5, J24.6, J24.7; no longer JP16.1, JP16.2, JP16.3, JP16.4, JP16.5, JP16.6, JP61.1
- net N$18: now also J25.1, J25.2, J25.3, J25.4, J25.5, J25.6, J25.7; no longer JP4.1, JP4.2, JP4.3, JP4.4, JP4.5, JP4.6, JP62.1
- net N$19: now also J26.1, J26.2, J26.3, J26.4, J26.5, J26.6, J26.7; no longer JP17.1, JP17.2, JP17.3, JP17.4, JP17.5, JP17.6, JP63.1
- net N$2: now also J9.1, J9.2, J9.3, J9.4, J9.5, J9.6, J9.7; no longer JP31.1, JP31.2, JP31.3, JP31.4, JP31.5, JP31.6, JP96.1
- net N$20: now also J27.1, J27.2, J27.3, J27.4, J27.5, J27.6, J27.7; no longer JP18.1, JP18.2, JP18.3, JP18.4, JP18.5, JP18.6, JP34.1
- net N$21: now also J28.1, J28.2, J28.3, J28.4, J28.5, J28.6, J28.7; no longer JP19.1, JP19.2, JP19.3, JP19.4, JP19.5, JP19.6, JP35.1
- net N$22: now also J29.1, J29.2, J29.3, J29.4, J29.5, J29.6, J29.7; no longer JP20.1, JP20.2, JP20.3, JP20.4, JP20.5, JP20.6, JP36.1
- net N$23: now also J30.1, J30.2, J30.3, J30.4, J30.5, J30.6, J30.7; no longer JP47.1, JP47.2, JP47.3, JP47.4, JP47.5, JP47.6, JP99.1
- net N$24: now also J31.1, J31.2, J31.3, J31.4, J31.5, J31.6, J31.7; no longer JP100.1, JP64.1, JP64.2, JP64.3, JP64.4, JP64.5, JP64.6
- net N$26: now also J32.1, J32.2, J32.3, J32.4, J32.5, J32.6, J32.7; no longer JP101.1, JP65.1, JP65.2, JP65.3, JP65.4, JP65.5, JP65.6
- net N$27: now also J33.1, J33.2, J33.3, J33.4, J33.5, J33.6, J33.7; no longer JP21.1, JP21.2, JP21.3, JP21.4, JP21.5, JP21.6, JP37.1
- net N$28: now also J34.1, J34.2, J34.3, J34.4, J34.5, J34.6, J34.7; no longer JP22.1, JP22.2, JP22.3, JP22.4, JP22.5, JP22.6, JP38.1
- net N$29: now also J35.1, J35.2, J35.3, J35.4, J35.5, J35.6, J35.7; no longer JP23.1, JP23.2, JP23.3, JP23.4, JP23.5, JP23.6, JP39.1
- net N$3: now also J10.1, J10.2, J10.3, J10.4, J10.5, J10.6, J10.7; no longer JP32.1, JP32.2, JP32.3, JP32.4, JP32.5, JP32.6, JP97.1
- net N$30: now also J36.1, J36.2, J36.3, J36.4, J36.5, J36.6, J36.7; no longer JP24.1, JP24.2, JP24.3, JP24.4, JP24.5, JP24.6, JP40.1
- net N$31: now also J37.1, J37.2, J37.3, J37.4, J37.5, J37.6, J37.7; no longer JP25.1, JP25.2, JP25.3, JP25.4, JP25.5, JP25.6, JP41.1
- net N$32: now also J38.1, J38.2, J38.3, J38.4, J38.5, J38.6, J38.7; no longer JP26.1, JP26.2, JP26.3, JP26.4, JP26.5, JP26.6, JP42.1
- net N$33: now also J39.1, J39.2, J39.3, J39.4, J39.5, J39.6, J39.7; no longer JP27.1, JP27.2, JP27.3, JP27.4, JP27.5, JP27.6, JP43.1
- net N$34: now also J40.1, J40.2, J40.3, J40.4, J40.5, J40.6, J40.7; no longer JP102.1, JP66.1, JP66.2, JP66.3, JP66.4, JP66.5, JP66.6
- net N$35: now also J41.1, J41.2, J41.3, J41.4, J41.5, J41.6, J41.7; no longer JP28.1, JP28.2, JP28.3, JP28.4, JP28.5, JP28.6, JP44.1
- net N$36: now also J42.1, J42.2, J42.3, J42.4, J42.5, J42.6, J42.7; no longer JP29.1, JP29.2, JP29.3, JP29.4, JP29.5, JP29.6, JP45.1
- net N$37: now also J43.1, J43.2, J43.3, J43.4, J43.5, J43.6, J43.7; no longer JP30.1, JP30.2, JP30.3, JP30.4, JP30.5, JP30.6, JP46.1
- net N$38: now also J44.1, J44.2, J44.3, J44.4, J44.5, J44.6, J44.7; no longer JP103.1, JP67.1, JP67.2, JP67.3, JP67.4, JP67.5, JP67.6
- net N$39: now also J45.1, J45.2, J45.3, J45.4, J45.5, J45.6, J45.7; no longer JP104.1, JP68.1, JP68.2, JP68.3, JP68.4, JP68.5, JP68.6
- net N$4: now also J11.1, J11.2, J11.3, J11.4, J11.5, J11.6, J11.7; no longer JP33.1, JP33.2, JP33.3, JP33.4, JP33.5, JP33.6, JP98.1
- net N$41: now also J47.1, J47.2, J47.3, J47.4, J47.5, J47.6, J47.7; no longer JP105.1, JP69.1, JP69.2, JP69.3, JP69.4, JP69.5, JP69.6
- net N$46: now also J50.1, J50.2, J50.3, J50.4, J50.5, J50.6, J50.7; no longer JP106.1, JP70.1, JP70.2, JP70.3, JP70.4, JP70.5, JP70.6
- net N$47: now also J51.1, J51.2, J51.3, J51.4, J51.5, J51.6, J51.7; no longer JP107.1, JP71.1, JP71.2, JP71.3, JP71.4, JP71.5, JP71.6
- net N$48: now also J52.1, J52.2, J52.3, J52.4, J52.5, J52.6, J52.7; no longer JP108.1, JP72.1, JP72.2, JP72.3, JP72.4, JP72.5, JP72.6
- net N$49: now also J53.1, J53.2, J53.3, J53.4, J53.5, J53.6, J53.7; no longer JP109.1, JP73.1, JP73.2, JP73.3, JP73.4, JP73.5, JP73.6
- net N$5: now also J12.1, J12.2, J12.3, J12.4, J12.5, J12.6, J12.7; no longer JP3.1, JP3.2, JP3.3, JP3.4, JP3.5, JP3.6, JP49.1
- net N$50: now also J54.1, J54.2, J54.3, J54.4, J54.5, J54.6, J54.7; no longer JP74.1, JP74.2, JP74.3, JP74.4, JP74.5, JP74.6, JP85.1
- net N$51: now also J55.1, J55.2, J55.3, J55.4, J55.5, J55.6, J55.7; no longer JP75.1, JP75.2, JP75.3, JP75.4, JP75.5, JP75.6, JP86.1
- net N$52: now also J56.1, J56.2, J56.3, J56.4, J56.5, J56.6, J56.7; no longer JP76.1, JP76.2, JP76.3, JP76.4, JP76.5, JP76.6, JP87.1
- net N$53: now also J57.1, J57.2, J57.3, J57.4, J57.5, J57.6, J57.7; no longer JP77.1, JP77.2, JP77.3, JP77.4, JP77.5, JP77.6, JP88.1
- net N$54: now also J58.1, J58.2, J58.3, J58.4, J58.5, J58.6, J58.7; no longer JP78.1, JP78.2, JP78.3, JP78.4, JP78.5, JP78.6, JP89.1
- net N$55: now also J59.1, J59.2, J59.3, J59.4, J59.5, J59.6, J59.7; no longer JP79.1, JP79.2, JP79.3, JP79.4, JP79.5, JP79.6, JP90.1
- net N$56: now also J60.1, J60.2, J60.3, J60.4, J60.5, J60.6; no longer JP80.1, JP80.2, JP80.3, JP80.4, JP80.5, JP80.6, JP91.1
- net N$6: now also J13.1, J13.2, J13.3, J13.4, J13.5, J13.6, J13.7; no longer JP5.1, JP5.2, JP5.3, JP5.4, JP5.5, JP5.6, JP50.1
- net N$7: now also J14.1, J14.2, J14.3, J14.4, J14.5, J14.6, J14.7; no longer JP51.1, JP6.1, JP6.2, JP6.3, JP6.4, JP6.5, JP6.6
- net N$8: now also J15.1, J15.2, J15.3, J15.4, J15.5, J15.6, J15.7; no longer JP52.1, JP7.1, JP7.2, JP7.3, JP7.4, JP7.5, JP7.6
- net N$9: now also J16.1, J16.2, J16.3, J16.4, J16.5, J16.6, J16.7; no longer JP53.1, JP8.1, JP8.2, JP8.3, JP8.4, JP8.5, JP8.6
