File: MX4-7-9/MX4-7-9-ESP12.brd (EAGLE design)
At the start: 82.8 x 59.2 mm, 67 parts, among them J1 DCJ0202, X2 ESP-12E

Commit message: Silkscreen text fixes
Silkscreen text fixes
Parts:
- moved RX 1.27 mm to (71.1, 23.5)
- moved TX 1.27 mm to (71.1, 26.0)
Routing:
- net N$1: track 105.4 -> 104.1 mm
- net N$2: track 87.3 -> 86.6 mm
