File: MX2-7-6/Protoboard MX2-7-6-ESP12.brd (EAGLE design)
At the start: 54.4 x 59.6 mm, 52 parts, among them X1 ESP-12E

Commit message: Silkscreen text fixes
Silkscreen text fixes
Other:
- board text added: "MX 2-7-6 rev 0"
- board text removed: "mx2-7-6-esp12-rev0"
